File: Ctrl-Project/P-channel.kicad_sch (KiCad schematic)
At the start: 7 parts, among them M1 Motor_DC, Q1 FQP27P06, U1 MC1458

Commit message: more project setup
Connections:
- net at RV1.1: now also RV1.2, RV2.3
Changed lines of the file:
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@@
   (junction (at 88.9 67.31) (diameter 0) (color 0 0 0 0)
+  )
+  (junction (at 25.4 64.77) (diameter 0) (color 0 0 0 0)
   )
   (junction (at 43.18 67.31) (diameter 0) (color 0 0 0 0)
@@
     (stroke (width 0) (type default) (color 0 0 0 0))
   )
+  (wire (pts (xy 25.4 64.77) (xy 25.4 67.31))
+    (stroke (width 0) (type default) (color 0 0 0 0))
+  )
